File: PDU_Control_Board.kicad_pcb (KiCad board)
At the start: 4 copper layers, 198 parts, among them J1 Current_Sensor, J10 Precharge_2, J11 Shunt_2, J12 VIN_Enable, J13 1-776087-1, J2 Shunt_1, J20 VDC_OUT2, J21 VDC_OUT1, J22 VDC_IN, J3 SWD, J4 Precharge_1, J5 Precharge_2, J6 Shunt_2, J7 VIN_Enable, J8 Precharge_1, J9 Shunt_1, Q1 BSP75N, Q10 BC817, Q2 BSP75N, Q3 BSP75N, Q4 BSP75N, Q5 BSP75N, Q6 BC817, Q7 BC817, Q8 BC817, Q9 BC817, U1 LMV321, U2 APM32F405xG, U3 LMV321, U4 LMV321, U5 LMV321, U6 LMV321, Y2 X322516MOB4SI

Commit message: VER1.0: сделал отвязанное измерение напряжения
Parts:
- removed R35, R36, R37, R41, R42, R43, R44, R45, R49, R50, R51, R52, R53, R54, R57, R58, R59, R60, R61, R62: 249k, Resistor_SMD:R_1206_3216Metric
- removed R38, R46, R55, R63: 4.99k, Resistor_SMD:R_0805_2012Metric_Pad1.20x1.40mm_HandSolder
- added C47: 0.1u, Capacitor_SMD:C_0805_2012Metric_Pad1.18x1.45mm_HandSolder, F.Cu at (256.3, 226.1)
- added C48: 2.2u, Capacitor_SMD:C_0805_2012Metric_Pad1.18x1.45mm_HandSolder, F.Cu at (256.3, 229.1)
- added C49: 56p, Capacitor_SMD:C_0805_2012Metric_Pad1.18x1.45mm_HandSolder, F.Cu at (256.3, 232.1)
- added C50: 2.2u, Capacitor_SMD:C_0805_2012Metric_Pad1.18x1.45mm_HandSolder, F.Cu at (256.3, 235.1)
- added C51: 0.1u, Capacitor_SMD:C_0805_2012Metric_Pad1.18x1.45mm_HandSolder, F.Cu at (256.3, 238.1)
- added C52: 56p, Capacitor_SMD:C_0805_2012Metric_Pad1.18x1.45mm_HandSolder, F.Cu at (256.3, 241.1)
- added C53: 2.2u, Capacitor_SMD:C_0805_2012Metric_Pad1.18x1.45mm_HandSolder, F.Cu at (261.1, 226.1)
- added C54: 0.1u, Capacitor_SMD:C_0805_2012Metric_Pad1.18x1.45mm_HandSolder, F.Cu at (261.1, 229.1)
- added C55: 2.2u, Capacitor_SMD:C_0805_2012Metric_Pad1.18x1.45mm_HandSolder, F.Cu at (261.1, 232.1)
- added C56: 0.1u, Capacitor_SMD:C_0805_2012Metric_Pad1.18x1.45mm_HandSolder, F.Cu at (261.1, 235.1)
- added C57: 56p, Capacitor_SMD:C_0805_2012Metric_Pad1.18x1.45mm_HandSolder, F.Cu at (261.1, 238.1)
- added C58: 2.2u, Capacitor_SMD:C_0805_2012Metric_Pad1.18x1.45mm_HandSolder, F.Cu at (261.1, 241.1)
- added C59: 0.1u, Capacitor_SMD:C_0805_2012Metric_Pad1.18x1.45mm_HandSolder, F.Cu at (265.9, 226.1)
- added C60: 2.2u, Capacitor_SMD:C_0805_2012Metric_Pad1.18x1.45mm_HandSolder, F.Cu at (265.9, 229.1)
- added C61: 0.1u, Capacitor_SMD:C_0805_2012Metric_Pad1.18x1.45mm_HandSolder, F.Cu at (265.9, 232.1)
- added D34: NSI1311, Package_SO:SOIC-8_7.5x5.85mm_P1.27mm, F.Cu at (435.4, 334.9)
- added D35: NSI1311, Package_SO:SOIC-8_7.5x5.85mm_P1.27mm, F.Cu at (435.4, 342.3)
- added D36: NSI1311, Package_SO:SOIC-8_7.5x5.85mm_P1.27mm, F.Cu at (435.4, 349.7)
- added D37: WRB2403S-3WR2, MORNSUN:WRB_S-3WR2, F.Cu at (436.4, 357.7)
- added D38: LED_Small, LED_SMD:LED_0805_2012Metric, F.Cu at (320.9, 311.4)
- added D39: LED_Small, LED_SMD:LED_0805_2012Metric, F.Cu at (320.9, 314.5)
- added R86: 120, Resistor_SMD:R_0805_2012Metric_Pad1.20x1.40mm_HandSolder, F.Cu at (261.9, 244.1)
- added R87: 240, Resistor_SMD:R_1206_3216Metric, F.Cu at (256.7, 244.3)
- added R88: 47k, Resistor_SMD:R_1206_3216Metric, F.Cu at (256.7, 247.6)
- added R89: 47k, Resistor_SMD:R_1206_3216Metric, F.Cu at (256.7, 250.9)
- C29, C30, C34, C35, C38, C8: value 4700p -> 56p
- J1: footprint Connector_Molex:Molex_Mini-Fit_Jr_5569-04A2_2x02_P4.20mm_Horizontal -> Connector_Molex:Molex_Mini-Fit_Jr_5566-04A_2x02_P4.20mm_Vertical
- R14, R30, R31, R47, R48, R64: value 3.74k -> 1k
- R15, R16, R23, R24: value 249k -> 47k
- R17, R25: value 249k -> 120; footprint Resistor_SMD:R_1206_3216Metric -> Resistor_SMD:R_0805_2012Metric_Pad1.20x1.40mm_HandSolder
- R18, R27: value 249k -> 240
- R19, R20, R26, R28: value 249k -> 1k; footprint Resistor_SMD:R_1206_3216Metric -> Resistor_SMD:R_0805_2012Metric_Pad1.20x1.40mm_HandSolder
- R21, R29: value 4.99k -> 1k
- R33, R34: value 249k -> 330; footprint Resistor_SMD:R_1206_3216Metric -> Resistor_SMD:R_0805_2012Metric_Pad1.20x1.40mm_HandSolder
- moved J20 226.0 mm to (450.6, 149.2)
- moved R32 163.0 mm to (191.8, 218.8)
- moved J21 161.0 mm to (450.5, 219.2)
- moved J13 135.5 mm to (335.0, 358.1), turned to 0 degrees
- moved J1 129.6 mm to (449.8, 324.6), turned to 180 degrees
- moved J22 127.9 mm to (450.5, 289.2)
- moved D25 112.4 mm to (279.6, 232.1)
- moved D26 112.4 mm to (279.6, 213.8)
- moved D27 112.4 mm to (279.6, 195.6)
- moved R81 112.4 mm to (279.6, 241.6)
- moved R82 112.4 mm to (279.6, 223.3)
- moved R83 112.4 mm to (279.6, 205.1)
- moved D2 112.3 mm to (324.2, 343.8), turned to -90 degrees
- moved C17 108.4 mm to (328.6, 340.0), turned to 180 degrees
- moved R6 107.0 mm to (324.2, 340.0), turned to 0 degrees
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Connections:
- C21 pad 1: +3.3V -> +3.3VA
- C21 pad 2: GND -> GNDA
- C22 pad 1: +3.3V -> +3.3VA
- C22 pad 2: GND -> GNDA
- C23 pad 2: GND -> GNDA
- C27 pad 2: GND -> GNDA
- C28 pad 2: GND -> GNDA
- C29 pad 1: Net-(C29-Pad1) -> Net-(U1--)
- C30 pad 1: GND -> GNDA
- C30 pad 2: Net-(C30-Pad2) -> Net-(U3-+)
- C31 pad 1: +3.3V -> +3.3VA
- C31 pad 2: GND -> GNDA
- C32 pad 2: GND -> GNDA
- C34 pad 1: Net-(C34-Pad1) -> Net-(U3--)
- C35 pad 1: GND -> GNDA
- C35 pad 2: Net-(C35-Pad2) -> Net-(U5-+)
- C36 pad 1: +3.3V -> +3.3VA
- C36 pad 2: GND -> GNDA
- C37 pad 2: GND -> GNDA
- C38 pad 1: Net-(C38-Pad1) -> Net-(U5--)
- C44 pad 1: +3.3V -> +3.3VA
- C44 pad 2: GND -> GNDA
- C45 pad 2: GND -> GNDA
- C46 pad 2: GND -> GNDA
- C8 pad 1: GND -> GNDA
- C8 pad 2: Net-(C8-Pad2) -> Net-(U1-+)
- D17 pad 1: GND -> GNDA
- D17 pad 2: +3.3V -> +3.3VA
- D18 pad 1: GND -> GNDA
- D18 pad 2: +3.3V -> +3.3VA
- D25 pad 1: VDC_OUT2_N -> GNDPWR
- D26 pad 1: VDC_OUT1_N -> GNDPWR
- D27 pad 1: VDC_IN_N -> GNDPWR
- D28 pad 1: GND -> GNDA
- D28 pad 2: +3.3V -> +3.3VA
- D5 pad 1: GND -> GNDA
- D5 pad 2: +3.3V -> +3.3VA
- R14 pad 1: GND -> GNDA
- R14 pad 2: Net-(C8-Pad2) -> Net-(U1-+)
- R15 pad 1: VDC_IN_P -> Net-(R15-Pad1)
- R15 pad 2: Net-(R15-Pad2) -> VDC_OUT1
- R16 pad 1: Net-(R15-Pad2) -> Net-(R16-Pad1)
- R16 pad 2: Net-(R16-Pad2) -> Net-(R15-Pad1)
- R17 pad 1: Net-(R16-Pad2) -> Net-(D35-VIN)
- R17 pad 2: Net-(R17-Pad2) -> Net-(R16-Pad1)
- R18 pad 1: Net-(R17-Pad2) -> GNDPWR
- R18 pad 2: Net-(R18-Pad2) -> Net-(R16-Pad1)
- R19 pad 1: Net-(R18-Pad2) -> Net-(D35-OUTP)
- R19 pad 2: Net-(R19-Pad2) -> Net-(U3-+)
- R20 pad 1: Net-(R19-Pad2) -> Net-(D35-OUTN)
- R20 pad 2: Net-(C8-Pad2) -> Net-(U3--)
- R21 pad 1: Net-(C8-Pad2) -> Net-(D34-OUTP)
- R23 pad 1: VDC_IN_N -> Net-(R23-Pad1)
- R23 pad 2: Net-(R23-Pad2) -> VDC_OUT1
- R24 pad 1: Net-(R23-Pad2) -> Net-(R24-Pad1)
- R24 pad 2: Net-(R24-Pad2) -> Net-(R23-Pad1)
- R25 pad 1: Net-(R24-Pad2) -> Net-(D36-VIN)
- R25 pad 2: Net-(R25-Pad2) -> Net-(R24-Pad1)
- R26 pad 1: Net-(R25-Pad2) -> Net-(D36-OUTP)
- R26 pad 2: Net-(R26-Pad2) -> Net-(U5-+)
- R27 pad 1: Net-(R26-Pad2) -> GNDPWR
- R27 pad 2: Net-(R27-Pad2) -> Net-(R24-Pad1)
- R28 pad 1: Net-(R27-Pad2) -> Net-(D36-OUTN)
- R28 pad 2: Net-(C29-Pad1) -> Net-(U5--)
- R29 pad 1: Net-(C29-Pad1) -> Net-(D34-OUTN)
- R30 pad 1: Net-(C29-Pad1) -> Net-(U1--)
- R31 pad 1: GND -> GNDA
- R31 pad 2: Net-(C30-Pad2) -> Net-(U3-+)
- R32 pad 2: Net-(R32-Pad2) -> unconnected-(R32-Pad2)
- R33 pad 1: Net-(R32-Pad2) -> Net-(U2-PE8)
- R33 pad 2: Net-(R33-Pad2) -> Net-(D38-A)
- R34 pad 1: Net-(R33-Pad2) -> Net-(U2-PE9)
- R40 pad 1: VDC_OUT1_N -> unconnected-(R40-Pad1)
- R40 pad 2: Net-(R40-Pad2) -> unconnected-(R40-Pad2)
- R47 pad 1: Net-(C34-Pad1) -> Net-(U3--)
- R48 pad 1: GND -> GNDA
- R48 pad 2: Net-(C35-Pad2) -> Net-(U5-+)
- R64 pad 1: Net-(C38-Pad1) -> Net-(U5--)
- R81 pad 1: VDC_OUT2_P -> VDC_OUT2
- R82 pad 1: VDC_OUT1_P -> VDC_OUT1
- R83 pad 1: VDC_IN_P -> VDC_IN
- R9 pad 2: GND -> GNDA
- U1 pad 2: GND -> GNDA
- U1 pad 5: +3.3V -> +3.3VA
- U2 pad 39: unconnected-(U2-PE8-Pad39) -> Net-(U2-PE8)
- U2 pad 40: unconnected-(U2-PE9-Pad40) -> Net-(U2-PE9)
- U3 pad 2: GND -> GNDA
- U3 pad 5: +3.3V -> +3.3VA
- U4 pad 2: GND -> GNDA
- U4 pad 5: +3.3V -> +3.3VA
- U5 pad 5: +3.3V -> +3.3VA
- U6 pad 2: GND -> GNDA
- U6 pad 5: +3.3V -> +3.3VA
Routing:
- net Shunt_1: track 21.4 -> 0.00 mm
- net ~{Precharge_2_ON}: track 20.8 -> 0.00 mm
- net Precharge_2: track 20.2 -> 0.00 mm
- net ~{Shunt_2_ON}: track 19.6 -> 0.00 mm
- net ~{Shunt_1_ON}: track 19.6 -> 0.00 mm
- net Shunt_2: track 19.0 -> 0.00 mm
- net ~{Precharge_1_ON}: track 20.0 -> 8.32 mm
- net VIN_Enable: track 19.4 -> 8.11 mm
- net ~{VIN_Enable_ON}: track 18.8 -> 7.86 mm
- net VDC_IN_SENSE: track 8.12 -> 3.74 mm
- net Current_SENSE: track 6.30 -> 1.93 mm
- net VDC_OUT2_SENSE: track 6.34 -> 2.53 mm
- net VDC_OUT1_SENSE: track 6.36 -> 3.15 mm

Commit message: VER1.0: обрезал плату
Parts:
- R33, R34: value 330 -> 1k
- moved R89 217.1 mm to (455.8, 337.5)
- moved R88 214.1 mm to (451.0, 337.5)
- moved C57 213.0 mm to (443.0, 349.0), turned to 90 degrees
- moved C49 212.8 mm to (443.0, 334.2), turned to 90 degrees
- moved R87 212.5 mm to (449.5, 333.8), turned to -90 degrees
- moved D27 212.1 mm to (462.0, 303.8), turned to -90 degrees
- moved C52 212.1 mm to (443.0, 341.8), turned to 90 degrees
- moved U5 211.6 mm to (421.2, 349.8)
- moved R83 210.2 mm to (462.0, 309.5), turned to 90 degrees
- moved R86 205.7 mm to (446.2, 335.2)
- moved C35 204.7 mm to (421.2, 352.5), turned to 0 degrees
- moved R48 202.7 mm to (421.2, 354.8), turned to 0 degrees
- moved R28 202.5 mm to (425.8, 348.2)
- moved R81 196.5 mm to (462.0, 168.5), turned to 90 degrees
- moved D25 195.2 mm to (462.0, 162.8), turned to -90 degrees
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Connections:
- D37 pad 1: unconnected-(D37-GND-Pad1) -> GND
- D37 pad 2: unconnected-(D37-Vin-Pad2) -> Net-(D37-Vin)
- D37 pad 6: unconnected-(D37-+Vo-Pad6) -> Net-(D37-+Vo)
- D37 pad 7: unconnected-(D37-0V-Pad7) -> Net-(D37-0V)
- J20 pad 1: VDC_OUT2_P -> VDC_IN
- J20 pad 2: VDC_OUT2_N -> GNDPWR
- J21 pad 1: VDC_OUT1_P -> VDC_OUT1
- J21 pad 2: VDC_OUT1_N -> GNDPWR
- J22 pad 1: VDC_IN_P -> VDC_OUT2
- J22 pad 2: VDC_IN_N -> GNDPWR
- R23 pad 2: VDC_OUT1 -> VDC_OUT2
Other:
- board outline added: 165.5 x 233.5 mm

Commit message: VER1.0: разместил все компоненты на плате
Parts:
- removed R32, R40: 249k, Resistor_SMD:R_1206_3216Metric
- added C62: 1u, Capacitor_Tantalum_SMD:CP_EIA-6032-28_Kemet-C_Pad2.25x2.35mm_HandSolder, F.Cu at (421.0, 360.7)
- added C63: 10u, Capacitor_Tantalum_SMD:CP_EIA-7360-38_Kemet-E_Pad2.25x4.25mm_HandSolder, F.Cu at (414.7, 360.0)
- added C64: 100u, Capacitor_Tantalum_SMD:CP_EIA-3528-21_Kemet-B_Pad1.50x2.35mm_HandSolder, F.Cu at (448.9, 363.2)
- added C65: 10u, Capacitor_Tantalum_SMD:CP_EIA-3528-21_Kemet-B_Pad1.50x2.35mm_HandSolder, F.Cu at (448.9, 357.5)
- added H1: MountingHole_Pad, MountingHole:MountingHole_3.2mm_M3_Pad_Via, F.Cu at (305.3, 173.7)
- added J14: Resistor, Connector_Molex:Molex_Mini-Fit_Jr_5566-06A_2x03_P4.20mm_Vertical, F.Cu at (308.4, 157.2)
- added J15: GNDPWR, Connector_My:Mini-Fit_01x02_Vertical, F.Cu at (454.7, 360.2)
- added J16: VDC_OUT1_Relay, Connector_My:Mini-Fit_01x02_Vertical, F.Cu at (340.4, 243.6)
- added J17: VDC_OUT2_Rela, Connector_My:Mini-Fit_01x02_Vertical, F.Cu at (340.9, 174.0)
- added L1: 4.7u, Inductor_SMD:L_1812_4532Metric_Pad1.30x3.40mm_HandSolder, F.Cu at (418.5, 367.0)
- C47, C48, C50, C51, C53, C54, C55, C56, C58, C59, C60, C61: moved to B.Cu
- J20: value VDC_OUT2 -> VDC_IN
- J22: value VDC_IN -> VDC_OUT2
- moved C22 238.0 mm to (417.6, 342.4)
- moved C36 225.3 mm to (397.8, 363.2)
- moved C31 225.2 mm to (403.4, 350.5)
- moved C53 216.6 mm to (443.5, 342.9), turned to -90 degrees
- moved C48 215.2 mm to (443.5, 335.3), turned to -90 degrees
- moved C47 214.5 mm to (440.9, 335.3), turned to 90 degrees
- moved C59 214.4 mm to (440.9, 350.0), turned to 90 degrees
- moved C54 212.8 mm to (440.9, 342.9), turned to 90 degrees
- moved C58 212.4 mm to (443.5, 350.0), turned to -90 degrees
- moved C23 208.1 mm to (413.1, 339.3), turned to 0 degrees
- moved R21 207.8 mm to (422.3, 343.9)
- moved R29 207.8 mm to (422.3, 340.9)
- moved U1 207.2 mm to (417.7, 342.4)
- moved D5 206.8 mm to (409.1, 339.3), turned to 0 degrees
- moved R22 205.9 mm to (413.1, 341.8), turned to 180 degrees
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Connections:
- D37 pad 6: Net-(D37-+Vo) -> +3.3VP
- D37 pad 7: Net-(D37-0V) -> GNDPWR
- D37 pad 8: unconnected-(D37-CS-Pad8) -> Net-(D37-CS)
- J20 pad 2: GNDPWR -> VDC_IN
- J21 pad 2: GNDPWR -> VDC_OUT1
- J22 pad 2: GNDPWR -> VDC_OUT2
- U5 pad 2: GND -> GNDA
Other:
- board size 165.5 x 233.5 mm -> 170.1 x 233.5 mm

Commit message: VER1.0: трассировал все дорожки и полигоны
Parts:
- removed C1: 4.7u, Capacitor_SMD:C_0805_2012Metric_Pad1.18x1.45mm_HandSolder
- removed C2: 100n, Capacitor_SMD:C_0805_2012Metric_Pad1.18x1.45mm_HandSolder
- removed C3: 1u, Capacitor_SMD:C_0805_2012Metric_Pad1.18x1.45mm_HandSolder
- removed FB1: BLM21BD121SN1D, Inductor_SMD:L_0805_2012Metric_Pad1.15x1.40mm_HandSolder
- removed R1: 0, Resistor_SMD:R_0805_2012Metric_Pad1.20x1.40mm_HandSolder
- added C66: 22u, Capacitor_Tantalum_SMD:CP_EIA-7343-43_Kemet-X_Pad2.25x2.55mm_HandSolder, F.Cu at (274.3, 238.6)
- added C67: 2.2n, Capacitor_SMD:C_0805_2012Metric_Pad1.18x1.45mm_HandSolder, F.Cu at (295.4, 280.5)
- added C68: 47n, Capacitor_SMD:C_0805_2012Metric_Pad1.18x1.45mm_HandSolder, F.Cu at (287.8, 267.8)
- added C69: 10u, Capacitor_SMD:C_1210_3225Metric_Pad1.33x2.70mm_HandSolder, F.Cu at (277.4, 243.9)
- added C70: 330u, Capacitor_Tantalum_SMD:CP_EIA-6032-28_Kemet-C_Pad2.25x2.35mm_HandSolder, F.Cu at (291.3, 242.7)
- added C71: 22u, Capacitor_SMD:C_1210_3225Metric_Pad1.33x2.70mm_HandSolder, F.Cu at (295.1, 242.7)
- added D40: LED_Small, LED_SMD:LED_0805_2012Metric, F.Cu at (282.2, 322.2)
- added D41: K7805-1000R3, MORNSUN:K78xx-1000R3, F.Cu at (284.2, 242.7)
- added D42: LED_Small, LED_SMD:LED_0805_2012Metric, F.Cu at (291.3, 251.3)
- added H2: MountingHole_Pad, MountingHole:MountingHole_4.3mm_M4, F.Cu at (305.6, 320.8)
- added H3: MountingHole_Pad, MountingHole:MountingHole_4.3mm_M4, F.Cu at (304.8, 97.8)
- added H4: MountingHole_Pad, MountingHole:MountingHole_4.3mm_M4_Pad_Via, F.Cu at (145.0, 320.8)
- added H6: MountingHole_Pad, MountingHole:MountingHole_4.3mm_M4, F.Cu at (145.4, 97.8)
- added R32: 665, Resistor_SMD:R_0805_2012Metric_Pad1.20x1.40mm_HandSolder, F.Cu at (298.4, 277.5)
- added R35: DNP, Resistor_SMD:R_0805_2012Metric_Pad1.20x1.40mm_HandSolder, F.Cu at (295.4, 276.5)
- added R36: 1k, Resistor_SMD:R_0805_2012Metric_Pad1.20x1.40mm_HandSolder, F.Cu at (299.5, 280.5)
- added R37: 750, Resistor_SMD:R_0805_2012Metric_Pad1.20x1.40mm_HandSolder, F.Cu at (284.7, 322.2)
- added R38: 1.1k, Resistor_SMD:R_0805_2012Metric_Pad1.20x1.40mm_HandSolder, F.Cu at (291.3, 248.8)
- H1: footprint MountingHole:MountingHole_3.2mm_M3_Pad_Via -> MountingHole:MountingHole_4.3mm_M4_Pad_Via
- R33, R34: moved to B.Cu
- moved C25 169.3 mm to (151.4, 307.5)
- moved C26 169.3 mm to (151.4, 291.0)
- moved C33 169.3 mm to (151.4, 311.9)
- moved D15 169.3 mm to (143.9, 307.5)
- moved D16 169.3 mm to (151.4, 299.2)
- moved D19 169.3 mm to (144.2, 291.0)
- moved R13 169.3 mm to (143.9, 310.0)
- moved R75 169.3 mm to (144.2, 288.5)
- moved C24 169.3 mm to (151.4, 286.5)
- moved J15 166.8 mm to (295.0, 312.2)
- moved D3 166.2 mm to (173.5, 290.9)
- moved C10 166.2 mm to (184.3, 267.1)
- moved C11 166.2 mm to (184.3, 271.9)
- moved C12 166.2 mm to (183.0, 264.1)
- moved C14 166.2 mm to (174.5, 264.1)
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Connections:
- C17 pad 2: CAN1H -> CANH
- C20 pad 1: CAN1L -> CANL
- C21 pad 1: +3.3VA -> +3.3V
- C21 pad 2: GNDA -> GND
- C22 pad 1: +3.3VA -> +3.3V
- C22 pad 2: GNDA -> GND
- C23 pad 2: GNDA -> GND
- C27 pad 2: GNDA -> GND
- C28 pad 2: GNDA -> GND
- C30 pad 1: GNDA -> GND
- C31 pad 1: +3.3VA -> +3.3V
- C31 pad 2: GNDA -> GND
- C32 pad 2: GNDA -> GND
- C35 pad 1: GNDA -> GND
- C36 pad 1: +3.3VA -> +3.3V
- C36 pad 2: GNDA -> GND
- C37 pad 2: GNDA -> GND
- C44 pad 1: +3.3VA -> +3.3V
- C44 pad 2: GNDA -> GND
- C45 pad 2: GNDA -> GND
- C46 pad 2: GNDA -> GND
- C50 pad 1: GNDA -> GND
- C50 pad 2: +3.3VA -> +3.3V
- C51 pad 1: +3.3VA -> +3.3V
- C51 pad 2: GNDA -> GND
- C55 pad 1: GNDA -> GND
- C55 pad 2: +3.3VA -> +3.3V
- C56 pad 1: +3.3VA -> +3.3V
- C56 pad 2: GNDA -> GND
- C60 pad 1: GNDA -> GND
- C60 pad 2: +3.3VA -> +3.3V
- C61 pad 1: +3.3VA -> +3.3V
- C61 pad 2: GNDA -> GND
- C8 pad 1: GNDA -> GND
- D1 pad 6: CAN1L -> CANL
- D1 pad 7: CAN1H -> CANH
- D17 pad 1: GNDA -> GND
- D17 pad 2: +3.3VA -> +3.3V
- D18 pad 1: GNDA -> GND
- D18 pad 2: +3.3VA -> +3.3V
- D2 pad 1: CAN1H -> CANH
- D2 pad 2: CAN1L -> CANL
- D28 pad 1: GNDA -> GND
- D28 pad 2: +3.3VA -> +3.3V
- D34 pad 5: GNDA -> GND
- D34 pad 8: +3.3VA -> +3.3V
- D35 pad 5: GNDA -> GND
- D35 pad 8: +3.3VA -> +3.3V
- D36 pad 5: GNDA -> GND
- D36 pad 8: +3.3VA -> +3.3V
- D38 pad 1: GND -> Net-(D38-K)
- D39 pad 1: GND -> Net-(D39-K)
- D5 pad 1: GNDA -> GND
- D5 pad 2: +3.3VA -> +3.3V
- J1 pad 1: unconnected-(J1-Pin_1-Pad1) -> Crrent_Out
- J1 pad 2: unconnected-(J1-Pin_2-Pad2) -> GND
- J1 pad 3: unconnected-(J1-Pin_3-Pad3) -> +5V
- J1 pad 4: unconnected-(J1-Pin_4-Pad4) -> GND
- J13 pad 1: unconnected-(J13-Pad1) -> +24V
- J13 pad 16: unconnected-(J13-Pad16) -> GND
- J13 pad 2: unconnected-(J13-Pad2) -> CANL
- J13 pad 3: unconnected-(J13-Pad3) -> CANH
- R14 pad 1: GNDA -> GND
- R31 pad 1: GNDA -> GND
- R33 pad 1: Net-(U2-PE8) -> Net-(D38-K)
- R33 pad 2: Net-(D38-A) -> GND
- R34 pad 1: Net-(U2-PE9) -> Net-(D39-K)
- R34 pad 2: Net-(D39-A) -> GND
- R48 pad 1: GNDA -> GND
- R6 pad 1: CAN1L -> CANL
- R6 pad 2: CAN1H -> CANH
- R85 pad 1: Current -> Net-(R32-Pad1)
- R9 pad 2: GNDA -> GND
- U1 pad 2: GNDA -> GND
- U1 pad 5: +3.3VA -> +3.3V
- U2 pad 20: GNDA -> GND
- U2 pad 21: +3.3VA -> +3.3V
- U2 pad 22: +3.3VA -> +3.3V
- U2 pad 30: Current_SENSE -> VDC_OUT2_SENSE
- U2 pad 31: VDC_OUT2_SENSE -> VDC_OUT1_SENSE
- U2 pad 32: VDC_OUT1_SENSE -> VDC_IN_SENSE
- U2 pad 33: VDC_IN_SENSE -> Current_SENSE
- U2 pad 39: Net-(U2-PE8) -> unconnected-(U2-PE8-Pad39)
- U2 pad 40: Net-(U2-PE9) -> unconnected-(U2-PE9-Pad40)
- U2 pad 52: unconnected-(U2-PB13-Pad52) -> Net-(D38-A)
- U2 pad 57: unconnected-(U2-PD10-Pad57) -> Net-(D39-A)
- U2 pad 60: Shunt_2 -> unconnected-(U2-PD13-Pad60)
- U2 pad 61: ~{Shunt_2_ON} -> unconnected-(U2-PD14-Pad61)
- U2 pad 62: Precharge_2 -> Shunt_1
- U2 pad 63: ~{Precharge_2_ON} -> ~{Shunt_1_ON}
- U2 pad 64: Shunt_1 -> Shunt_2
- U2 pad 65: ~{Shunt_1_ON} -> ~{Shunt_2_ON}
- U2 pad 66: Precharge_1 -> Precharge_2
- U2 pad 67: ~{Precharge_1_ON} -> ~{Precharge_2_ON}
- U2 pad 68: VIN_Enable -> Precharge_1
- U2 pad 69: ~{VIN_Enable_ON} -> ~{Precharge_1_ON}
- U2 pad 98: unconnected-(U2-PE1-Pad98) -> ~{VIN_Enable_ON}
- U3 pad 2: GNDA -> GND
- U3 pad 5: +3.3VA -> +3.3V
- U4 pad 2: GNDA -> GND
- U4 pad 5: +3.3VA -> +3.3V
- U5 pad 2: GNDA -> GND
- U5 pad 5: +3.3VA -> +3.3V
- U6 pad 2: GNDA -> GND
- U6 pad 5: +3.3VA -> +3.3V
Routing:
- net VDC_IN: track 0.00 -> 347.4 mm
- net VDC_OUT2: track 0.00 -> 203.6 mm
- net ~{Shunt_2_ON}: track 0.00 -> 202.8 mm
- net Shunt_2: track 0.00 -> 199.4 mm
- net ~{Shunt_1_ON}: track 0.00 -> 167.0 mm
- net Shunt_1: track 0.00 -> 155.3 mm
- net ~{Precharge_2_ON}: track 0.00 -> 155.1 mm
- net GND: track 0.00 -> 154.4 mm, vias 0 -> 101
- net Precharge_2: track 0.00 -> 133.1 mm
- net VDC_OUT1: track 0.00 -> 122.1 mm
- net Current_SENSE: track 1.93 -> 112.8 mm
- net VDC_OUT1_Relay: track 0.00 -> 109.7 mm
- net +24V: track 0.00 -> 105.6 mm, vias 0 -> 12
- net VDC_IN_SENSE: track 3.74 -> 101.1 mm
- net VDC_OUT2_SENSE: track 2.53 -> 99.3 mm
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- added copper zone on B.Cu, net +24V
- added copper zone on F.Cu, net +24V
- added copper zone on F.Cu, net +3.3V
- added copper zone on In1.Cu, net +3.3V
- added copper zone on In1.Cu, net +3.3VP
- added copper zone on F.Cu, net +5V
- added copper zone on B.Cu, net GND
- added copper zone on F.Cu, net GND
- added copper zone on In2.Cu, net GND
- added copper zone on In2.Cu, net GNDPWR
- added copper zone on F.Cu, net Net-(D37-Vin)
Other:
- board size 170.1 x 233.5 mm -> 170.4 x 233.5 mm
