File: PDU_Control_Board.kicad_pcb (KiCad board)
At the start: 4 copper layers, 237.7 x 87.4 mm, 211 parts, among them J1 Current_Sensor, J10 Precharge_2, J11 Shunt_2, J12 VIN_Enable, J13 To_Main_Connector, J2 Shunt_1, J20 VDC_IN, J21 VDC_OUT1, J22 VDC_OUT2, J3 SWD, J4 Precharge_1, J5 Precharge_2, J6 Shunt_2, J7 VIN_Enable, J8 Precharge_1, J9 Shunt_1, Q1 BSP75N, Q10 BC817, Q2 BSP75N, Q3 BSP75N, Q4 BSP75N, Q5 BSP75N, Q6 BC817, Q7 BC817, Q8 BC817, Q9 BC817, U1 LMV321, U2 APM32F405xG, U3 LMV321, U4 LMV321, U5 LMV321, U6 LMV321, Y2 X322516MOB4SI

Commit message: VER3.0: плата готова
Parts:
- added C1: 100n, Capacitor_SMD:C_0805_2012Metric_Pad1.18x1.45mm_HandSolder, B.Cu at (304.2, 213.4)
- added C2: 1u, Capacitor_SMD:C_0805_2012Metric_Pad1.18x1.45mm_HandSolder, B.Cu at (315.6, 221.6)
- added C3: 100n, Capacitor_SMD:C_0805_2012Metric_Pad1.18x1.45mm_HandSolder, B.Cu at (316.9, 215.9)
- added C72: 1u, Capacitor_SMD:C_0805_2012Metric_Pad1.18x1.45mm_HandSolder, B.Cu at (310.5, 221.6)
- added C73: 4.7u, Capacitor_SMD:C_0805_2012Metric_Pad1.18x1.45mm_HandSolder, B.Cu at (304.2, 215.9)
- added C74: 100n, Capacitor_SMD:C_0805_2012Metric_Pad1.18x1.45mm_HandSolder, B.Cu at (316.9, 213.4)
- added C75: 100n, Capacitor_SMD:C_0805_2012Metric_Pad1.18x1.45mm_HandSolder, B.Cu at (310.5, 208.9)
- added G***: LOGO, Logo_My:EV_Tech, F.Cu at (365.1, 208.9)
- added G***: LOGO, Logo_My:High_Voltage, F.Cu at (444.5, 174.0)
- C68: moved to B.Cu
- R33, R34: moved to F.Cu
- moved R9 46.5 mm to (379.1, 229.9), turned to -90 degrees
- moved R13 45.2 mm to (259.7, 241.3), turned to 0 degrees
- moved R7 45.1 mm to (381.6, 229.9), turned to 90 degrees
- moved C27 43.4 mm to (376.6, 229.9), turned to -90 degrees
- moved R35 43.1 mm to (236.2, 194.3)
- moved C67 42.8 mm to (236.2, 198.8)
- moved J1 42.3 mm to (231.8, 194.8)
- moved D28 41.5 mm to (263.5, 199.4)
- moved R36 41.5 mm to (242.6, 198.8)
- moved R32 41.2 mm to (239.4, 197.5)
- moved C45 41.1 mm to (260.4, 200.7)
- moved D15 41.0 mm to (255.9, 241.3), turned to 180 degrees
- moved R84 40.2 mm to (257.2, 199.4), turned to 0 degrees
- moved C21 40.1 mm to (373.4, 229.9), turned to 90 degrees
- moved U4 40.1 mm to (373.4, 229.9), turned to -90 degrees
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Connections:
- J10 pad 1: +24V -> Net-(D22-A)
- J10 pad 2: Net-(D22-A) -> +24V
- J11 pad 1: +24V -> Net-(D21-A)
- J11 pad 2: Net-(D21-A) -> +24V
- J12 pad 1: +24V -> Net-(D20-A)
- J12 pad 2: Net-(D20-A) -> +24V
- J13 pad 2: +24V -> CANH
- J13 pad 3: CANH -> +24V
- J2 pad 1: +24V -> Net-(D6-A)
- J2 pad 2: Net-(D6-A) -> +24V
- J4 pad 1: +24V -> Net-(D7-A)
- J4 pad 2: Net-(D7-A) -> +24V
- J5 pad 1: +24V -> Net-(D4-A)
- J5 pad 2: Net-(D4-A) -> +24V
- J6 pad 1: +24V -> Net-(D8-A)
- J6 pad 2: Net-(D8-A) -> +24V
- J7 pad 1: +24V -> Net-(D13-A)
- J7 pad 2: Net-(D13-A) -> +24V
- J8 pad 1: +24V -> Net-(D24-A)
- J8 pad 2: Net-(D24-A) -> +24V
- J9 pad 1: +24V -> Net-(D23-A)
- J9 pad 2: Net-(D23-A) -> +24V
- U2 pad 30: VDC_OUT2_SENSE -> Current_SENSE
- U2 pad 31: VDC_OUT1_SENSE -> VDC_OUT2_SENSE
- U2 pad 32: VDC_IN_SENSE -> VDC_OUT1_SENSE
- U2 pad 33: Current_SENSE -> VDC_IN_SENSE
- U2 pad 60: unconnected-(U2-PD13-Pad60) -> Shunt_2
- U2 pad 61: unconnected-(U2-PD14-Pad61) -> ~{Shunt_2_ON}
- U2 pad 62: Shunt_1 -> Precharge_2
- U2 pad 63: ~{Shunt_1_ON} -> ~{Precharge_2_ON}
- U2 pad 64: Shunt_2 -> Shunt_1
- U2 pad 65: ~{Shunt_2_ON} -> ~{Shunt_1_ON}
- U2 pad 66: Precharge_2 -> Precharge_1
- U2 pad 67: ~{Precharge_2_ON} -> ~{Precharge_1_ON}
- U2 pad 68: Precharge_1 -> VIN_Enable
- U2 pad 69: ~{Precharge_1_ON} -> ~{VIN_Enable_ON}
- U2 pad 98: ~{VIN_Enable_ON} -> unconnected-(U2-PE1-Pad98)
Routing:
- net VDC_OUT2_SENSE: track 4.13 -> 122.3 mm
- net Current_SENSE: track 2.32 -> 102.1 mm
- net VDC_OUT1_SENSE: track 6.55 -> 106.1 mm
- net VDC_IN_SENSE: track 6.68 -> 89.9 mm
- net Shunt_2: track 16.2 -> 95.1 mm
- net VIN_Enable: track 0.00 -> 69.8 mm
- net ~{VIN_Enable_ON}: track 9.48 -> 78.8 mm
- net CANL: track 8.69 -> 72.7 mm
- net ~{Shunt_2_ON}: track 15.9 -> 79.8 mm
- net CANH: track 8.69 -> 69.5 mm
- net DC_Voltage_MCU: track 2.63 -> 57.9 mm
- net Precharge_2: track 11.5 -> 65.5 mm
- net +3.3V: track 74.5 -> 113.5 mm, vias 30 -> 35
- net ~{Precharge_2_ON}: track 17.2 -> 49.7 mm
- net ~{Precharge_1_ON}: track 18.4 -> 50.2 mm
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- added copper zone on In1.Cu, net +24V
- added copper zone on In1.Cu, net +3.3V
- added copper zone on F.Cu, net +3.3VP
- added copper zone on In2.Cu, net +3.3VP
- added copper zone on F.Cu, net +5V
- added copper zone on In2.Cu, net +5V
- added copper zone on B.Cu, net GNDPWR
- added copper zone on F.Cu, net GNDPWR
Other:
- board text added: "+24V"
- board text added: "+3.3V"
- board text added: "+5V"
- board text added: "Current Sensor"
- board text added: "Main Connector"
- board text added: "PDU Control Board VER1.0"
- board text added: "Precharge 1"
- board text added: "Precharge 2"
- board text added: "Shunt 1"
- board text added: "Shunt 2"
- board text added: "VDC_IN"
- board text added: "VDC_IN Enable"
- board text added: "VOUT 1"
- board text added: "VOUT 2"

Commit message: VER3.0: добавил шелкографию на заднюю сторону
Parts:
- added G***: LOGO, Logo_My:High_Voltage, B.Cu at (444.5, 174.0)
